Commit message: 加入elmo_gold

File: ethercat_motor_drive/description/ros2_control/motor_drive.ros2_control.xacro (robot description, xacro)
@@ -8,5 +8,5 @@
         <param name="control_frequency">100</param>
       </hardware>
-      <joint name="joint_1">
+      <joint name="joint_0">
         <state_interface name="position"/>
         <state_interface name="velocity"/>
@@ -22,4 +22,46 @@
         </ec_module>
       </joint>
+      <joint name="joint_1">
+        <state_interface name="position"/>
+        <state_interface name="velocity"/>
+        <state_interface name="effort"/>
+        <command_interface name="position"/>
+        <command_interface name="reset_fault"/>
+        <ec_module name="Maxon">
+          <plugin>ethercat_generic_plugins/EcCiA402Drive</plugin>
+          <param name="alias">0</param>
+          <param name="position">1</param>
+          <param name="mode_of_operation">8</param>
+          <param name="slave_config">$(find ethercat_motor_drive)/config/elmo_gold_config.yaml</param>
+        </ec_module>
+      </joint>
+      <joint name="joint_2">
+        <state_interface name="position"/>
+        <state_interface name="velocity"/>
+        <state_interface name="effort"/>
+        <command_interface name="position"/>
+        <command_interface name="reset_fault"/>
+        <ec_module name="Maxon">
+          <plugin>ethercat_generic_plugins/EcCiA402Drive</plugin>
+          <param name="alias">0</param>
+          <param name="position">2</param>
+          <param name="mode_of_operation">8</param>
+          <param name="slave_config">$(find ethercat_motor_drive)/config/elmo_gold_config.yaml</param>
+        </ec_module>
+      </joint>
+      <joint name="joint_3">
+        <state_interface name="position"/>
+        <state_interface name="velocity"/>
+        <state_interface name="effort"/>
+        <command_interface name="position"/>
+        <command_interface name="reset_fault"/>
+        <ec_module name="Maxon">
+          <plugin>ethercat_generic_plugins/EcCiA402Drive</plugin>
+          <param name="alias">0</param>
+          <param name="position">3</param>
+          <param name="mode_of_operation">8</param>
+          <param name="slave_config">$(find ethercat_motor_drive)/config/elmo_gold_config.yaml</param>
+        </ec_module>
+      </joint>
     </ros2_control>
   </xacro:macro>
